Commit message: 添加机械臂毕设

File: aliengo_description/xacro/robot.xacro (robot description, xacro)
@@ -114,5 +114,5 @@
         </collision>
     </link>
-    <joint name="camera_joint" type="fixed">
+    <!-- <joint name="camera_joint" type="fixed">
         <parent link="trunk"/>
         <child link="camera_link"/>
@@ -138,5 +138,5 @@
             </geometry>
         </collision>
-    </link>
+    </link> -->
     <joint name="laser_joint" type="fixed">
         <parent link="trunk"/>

File: aliengo_gazebo/launch/gazebo.xacro (robot description, xacro)
@@ -4,5 +4,5 @@
     <gazebo>
         <plugin name="gazebo_ros_control" filename="libgazebo_ros_control.so">
-            <robotNamespace>/laikago_gazebo</robotNamespace>
+            <!-- <robotNamespace>/laikago_gazebo</robotNamespace> -->
             <robotSimType>gazebo_ros_control/DefaultRobotHWSim</robotSimType>
         </plugin>
@@ -56,5 +56,5 @@
     </gazebo>
 	<!-- RGBD Plugin -->
-	<gazebo reference="camera_link">
+	<!-- <gazebo reference="camera_link">
 		<sensor name="camera_link_name" type="depth">
 			<update_rate>20</update_rate>
@@ -96,5 +96,5 @@
 			</plugin>
 		</sensor>
-	</gazebo>
+	</gazebo> -->
 	<!--3D LiDAR -->
 	<gazebo reference="laser_link">
